File: boards/Production/ODKB_Board.kicad_pcb (KiCad board)
At the start: 2 copper layers, 428 x 125.7 mm, 350 parts, among them J1 Conn_01x05_Male, J2 USB_B_Micro, J3 Conn_01x03_Male, SW1 ESC, SW10 Z, SW100 ENT, SW101 DEL, SW102 END, SW103 PGDN, SW104 =, SW11 WIN, SW12 F1, SW13 2, SW14 W, SW15 S, SW16 X, SW17 ALT, SW18 F2, SW19 3, SW2 `, SW20 E, SW21 D, SW22 C, SW23 F3, SW24 4, SW25 R, SW26 F, SW27 V, SW28 F4, SW29 5, SW3 TAB, SW30 T, SW31 G, SW32 B, SW33 F5, SW34 6, SW35 Y, SW36 H, SW37 N, SW38 F6, SW39 7, SW4 CAPS, SW40 U, SW41 J, SW42 M, SW43 SPC, SW44 F7, SW45 8, SW46 I, SW47 K, SW48 ,<, SW49 F8, SW5 LSHIFT, SW50 9, SW51 O, SW52 L, SW53 .>, SW54 F9, SW55 0, SW56 P, SW57 ;, SW58 /?, SW59 ALT, SW6 CTRL, SW60 F10, SW61 -, SW62 [, SW63 ', SW64 FN, SW65 F11, SW66 ], SW67 FXN, SW68 F12, SW69 BACKSPACE, SW7 1, SW70 \, SW71 ENTER, SW72 RSHIFT, SW73 CTRL, SW74 PRINT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

Commit message: gitignore
Parts:
- moved SW103 708.7 mm to (686.8, 299.7)
- moved SW83 695.4 mm to (686.8, 356.7)
- moved SW102 680.9 mm to (667.8, 299.7)
- moved SW101 666.3 mm to (648.8, 299.7)
- moved SW82 660.9 mm to (686.8, 280.7)
- moved SW76 653.3 mm to (648.8, 356.7)
- moved SW80 645.8 mm to (667.8, 356.7)
- moved SW79 617.9 mm to (667.8, 337.7)
- moved SW78 595.2 mm to (667.8, 280.7)
- moved SW75 440.1 mm to (648.8, 280.7)
- moved D110 0.31 mm to (347.3, 263.1)
Changed lines of the file:
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@@
   )
   (module Diode_THT:D_DO-15_P10.16mm_Horizontal (layer F.Cu)
-    (at 347 263 90)
+    (at 347.3 263.06 90)
     (descr "Diode, DO-15 series, Axial, Horizontal, pin pitch=10.16mm, , length*diameter=7.6*3.6mm^2, , http://www.diodes.com/_files/packages/DO-15.pdf")
     (tags "Diode DO-15 series Axial Horizontal pin pitch 10.16mm  length 7.6mm diameter 3.6mm")
@@
   )
   (module Button_Switch_Keyboard:SW_Cherry_MX1A_1.00u_PCB (layer F.Cu)
-    (at 257.490001 79.120001)
+    (at 648.75 280.7)
     (descr "Cherry MX keyswitch, MX1A, 1.00u, PCB mount, http://cherryamericas.com/wp-content/uploads/2014/12/mx_cat.pdf")
     (tags "cherry mx keyswitch MX1A 1.00u PCB")
@@
   )
   (module Button_Switch_Keyboard:SW_Cherry_MX1A_1.00u_PCB (layer F.Cu)
-    (at 27.090001 155.920001)
+    (at 648.75 356.7)
     (descr "Cherry MX keyswitch, MX1A, 1.00u, PCB mount, http://cherryamericas.com/wp-content/uploads/2014/12/mx_cat.pdf")
     (tags "cherry mx keyswitch MX1A 1.00u PCB")
@@
   )
   (module Button_Switch_Keyboard:SW_Cherry_MX1A_1.00u_PCB (layer F.Cu)
-    (at 123.090001 40.720001)
+    (at 667.75 280.7)
     (descr "Cherry MX keyswitch, MX1A, 1.00u, PCB mount, http://cherryamericas.com/wp-content/uploads/2014/12/mx_cat.pdf")
     (tags "cherry mx keyswitch MX1A 1.00u PCB")
@@
   )
   (module Button_Switch_Keyboard:SW_Cherry_MX1A_1.00u_PCB (layer F.Cu)
-    (at 112.59 66.46)
+    (at 667.75 337.7)
     (descr "Cherry MX keyswitch, MX1A, 1.00u, PCB mount, http://cherryamericas.com/wp-content/uploads/2014/12/mx_cat.pdf")
     (tags "cherry mx keyswitch MX1A 1.00u PCB")
@@
   )
   (module Button_Switch_Keyboard:SW_Cherry_MX1A_1.00u_PCB (layer F.Cu)
-    (at 84.690001 79.120001)
+    (at 667.75 356.7)
     (descr "Cherry MX keyswitch, MX1A, 1.00u, PCB mount, http://cherryamericas.com/wp-content/uploads/2014/12/mx_cat.pdf")
     (tags "cherry mx keyswitch MX1A 1.00u PCB")
@@
   )
   (module Button_Switch_Keyboard:SW_Cherry_MX1A_1.00u_PCB (layer F.Cu)
-    (at 46.290001 117.520001)
+    (at 686.75 280.7)
     (descr "Cherry MX keyswitch, MX1A, 1.00u, PCB mount, http://cherryamericas.com/wp-content/uploads/2014/12/mx_cat.pdf")
     (tags "cherry mx keyswitch MX1A 1.00u PCB")
@@
   )
   (module Button_Switch_Keyboard:SW_Cherry_MX1A_1.00u_PCB (layer F.Cu)
-    (at 27.090001 136.720001)
+    (at 686.75 356.7)
     (descr "Cherry MX keyswitch, MX1A, 1.00u, PCB mount, http://cherryamericas.com/wp-content/uploads/2014/12/mx_cat.pdf")
     (tags "cherry mx keyswitch MX1A 1.00u PCB")
@@
   )
   (module Button_Switch_Keyboard:SW_Cherry_MX1A_1.00u_PCB (layer F.Cu)
-    (at 27.090001 59.920001)
+    (at 648.75 299.7)
     (descr "Cherry MX keyswitch, MX1A, 1.00u, PCB mount, http://cherryamericas.com/wp-content/uploads/2014/12/mx_cat.pdf")
     (tags "cherry mx keyswitch MX1A 1.00u PCB")
@@
   )
   (module Button_Switch_Keyboard:SW_Cherry_MX1A_1.00u_PCB (layer F.Cu)
-    (at 46.290001 21.520001)
+    (at 667.75 299.7)
     (descr "Cherry MX keyswitch, MX1A, 1.00u, PCB mount, http://cherryamericas.com/wp-content/uploads/2014/12/mx_cat.pdf")
     (tags "cherry mx keyswitch MX1A 1.00u PCB")
@@
   )
   (module Button_Switch_Keyboard:SW_Cherry_MX1A_1.00u_PCB (layer F.Cu)
-    (at 27.090001 40.720001)
+    (at 686.75 299.7)
     (descr "Cherry MX keyswitch, MX1A, 1.00u, PCB mount, http://cherryamericas.com/wp-content/uploads/2014/12/mx_cat.pdf")
     (tags "cherry mx keyswitch MX1A 1.00u PCB")
